Commit message: changes to enable running of simulation with scarab

File: scarab_description/urdf/kobuki.urdf.xacro (robot description, xacro)
@@ -147,4 +147,20 @@
       </inertial>
     </link>
+    <!-- Kobuki's sensors -->
+    <joint name="gyro_joint" type="fixed">
+      <axis xyz="0 1 0"/>
+      <origin xyz="0.056 0.062 0.0202" rpy="0 0 0"/>
+      <parent link="base_link"/>
+      <child link="gyro_link"/>
+    </joint>
+    <link name="gyro_link">
+      <inertial>
+        <mass value="0.001"/>
+        <origin xyz="0 0 0" rpy="0 0 0"/>
+        <inertia ixx="0.0001" ixy="0" ixz="0"
+                 iyy="0.000001" iyz="0"
+                 izz="0.0001"/>
+      </inertial>
+    </link>
     <!-- Kobuki Gazebo simulation details -->
     <kobuki_sim/>

File: scarab_description/urdf/kobuki_gazebo.urdf.xacro (robot description, xacro)
@@ -44,11 +44,12 @@
         <leftJoint>wheel_right_joint</leftJoint>
         <rightJoint>wheel_left_joint</rightJoint>
+        <legacyMode>true</legacyMode>
         <wheelSeparation>0.230</wheelSeparation>
         <wheelDiameter>0.070</wheelDiameter>
         <torque>1.0</torque>
         <commandTopic>cmd_vel</commandTopic>
-        <odometryTopic>ground_truth/odom</odometryTopic>
-        <odometryFrame>ground_truth/odom</odometryFrame>
-        <robotBaseFrame>ground_truth/base_link</robotBaseFrame>
+        <odometryTopic>odom</odometryTopic>
+        <odometryFrame>odom</odometryFrame>
+        <robotBaseFrame>base_footprint</robotBaseFrame>
         <publishWheelJointState>false</publishWheelJointState>
         <wheelAcceleration>0</wheelAcceleration>
@@ -59,4 +60,16 @@
       </plugin>
     </gazebo>
+    <gazebo>
+      <plugin name="p3d_base_controller" filename="libgazebo_ros_p3d.so">
+        <alwaysOn>true</alwaysOn>
+        <updateRate>50.0</updateRate>
+        <bodyName>base_link</bodyName>
+        <topicName>ground_truth/state</topicName>
+        <gaussianNoise>0.01</gaussianNoise>
+        <frameName>world</frameName>
+        <xyzOffsets>0 0 0</xyzOffsets>
+        <rpyOffsets>0 0 0</rpyOffsets>
+      </plugin>
+    </gazebo>
   </xacro:macro>
 </robot>
