Commit message: enable multi-scarab gazebo simulations
1) added tf_prefix throughout scarab description files to avoid tf collisions
2) updated scarab_sim.launch file to work with update tf tree
3) added PERCH environment

File: scarab_description/urdf/hexagons.urdf.xacro (robot description, xacro)
@@ -9,11 +9,11 @@
   <!-- Xacro macros -->
   <!-- Pole macros -->
-  <xacro:macro name="stack_bottom_pole" params="parent number x_loc y_loc z_loc">
-    <joint name="pole_bottom_${number}_joint" type="fixed">
+  <xacro:macro name="stack_bottom_pole" params="parent prefix number x_loc y_loc z_loc">
+    <joint name="${prefix}/pole_bottom_${number}_joint" type="fixed">
       <origin xyz="${x_loc} ${y_loc} ${z_loc}" rpy="0 0 0"/>
       <parent link="${parent}"/>
-      <child link="pole_bottom_${number}_link"/>
-    </joint>
-    <link name="pole_bottom_${number}_link">
+      <child link="${prefix}/pole_bottom_${number}_link"/>
+    </joint>
+    <link name="${prefix}/pole_bottom_${number}_link">
       <visual>
         <origin xyz="0 0 0" rpy="0 0 0"/>
@@ -37,11 +37,11 @@
     </link>
   </xacro:macro>
-  <xacro:macro name="stack_middle_pole" params="parent number x_loc y_loc z_loc">
-    <joint name="pole_middle_${number}_joint" type="fixed">
+  <xacro:macro name="stack_middle_pole" params="parent prefix number x_loc y_loc z_loc">
+    <joint name="${prefix}/pole_middle_${number}_joint" type="fixed">
       <origin xyz="${x_loc} ${y_loc} ${z_loc}" rpy="0 0 0" />
       <parent link="${parent}"/>
-      <child link="pole_middle_${number}_link"/>
-    </joint>
-    <link name="pole_middle_${number}_link">
+      <child link="${prefix}/pole_middle_${number}_link"/>
+    </joint>
+    <link name="${prefix}/pole_middle_${number}_link">
       <visual>
         <origin xyz="0 0 0" rpy="0 ${M_PI} 0"/>
@@ -65,11 +65,11 @@
     </link>
   </xacro:macro>
-  <xacro:macro name="stack_top_pole" params="parent number x_loc y_loc z_loc">
-    <joint name="pole_top_${number}_joint" type="fixed">
+  <xacro:macro name="stack_top_pole" params="parent prefix number x_loc y_loc z_loc">
+    <joint name="${prefix}/pole_top_${number}_joint" type="fixed">
       <origin xyz="${x_loc} ${y_loc} ${z_loc}" rpy="0 0 0"/>
       <parent link="${parent}"/>
-      <child link="pole_top_${number}_link"/>
-    </joint>
-    <link name="pole_top_${number}_link">
+      <child link="${prefix}/pole_top_${number}_link"/>
+    </joint>
+    <link name="${prefix}/pole_top_${number}_link">
       <visual>
         <origin xyz=" 0 0 0" rpy="0 0 0"/>
@@ -93,11 +93,11 @@
     </link>
   </xacro:macro>
-  <xacro:macro name="stack_3d_sensor_pole" params="parent number x_loc y_loc z_loc">
-    <joint name="pole_kinect_${number}_joint" type="fixed">
+  <xacro:macro name="stack_3d_sensor_pole" params="parent prefix number x_loc y_loc z_loc">
+    <joint name="${prefix}/pole_kinect_${number}_joint" type="fixed">
       <origin xyz="${x_loc} ${y_loc} ${z_loc}" rpy="0 0 0"/>
       <parent link="${parent}"/>
-      <child link="pole_kinect_${number}_link"/>
-    </joint>
-    <link name="pole_kinect_${number}_link">
+      <child link="${prefix}/pole_kinect_${number}_link"/>
+    </joint>
+    <link name="${prefix}/pole_kinect_${number}_link">
       <visual>
         <origin xyz="0 0 0" rpy="0 0 0"/>
@@ -127,17 +127,17 @@
     other, but there is no necessary reason to do so.
   -->
-  <xacro:macro name="stack_hexagons" params="parent">
-    <xacro:stack_bottom_pole parent="${parent}" number="0" x_loc= "0.120" y_loc= "0.082" z_loc="0.1028"/>
-    <xacro:stack_bottom_pole parent="${parent}" number="1" x_loc= "0.055" y_loc= "0.120" z_loc="0.1028"/>
-    <xacro:stack_bottom_pole parent="${parent}" number="2" x_loc="-0.055" y_loc= "0.120" z_loc="0.1028"/>
-    <xacro:stack_bottom_pole parent="${parent}" number="3" x_loc= "0.120" y_loc="-0.082" z_loc="0.1028"/>
-    <xacro:stack_bottom_pole parent="${parent}" number="4" x_loc= "0.055" y_loc="-0.120" z_loc="0.1028"/>
-    <xacro:stack_bottom_pole parent="${parent}" number="5" x_loc="-0.055" y_loc="-0.120" z_loc="0.1028"/>
-    <joint name="plate_bottom_joint" type="fixed">
+  <xacro:macro name="stack_hexagons" params="parent prefix">
+    <xacro:stack_bottom_pole parent="${parent}" prefix="${prefix}" number="0" x_loc= "0.120" y_loc= "0.082" z_loc="0.1028"/>
+    <xacro:stack_bottom_pole parent="${parent}" prefix="${prefix}" number="1" x_loc= "0.055" y_loc= "0.120" z_loc="0.1028"/>
+    <xacro:stack_bottom_pole parent="${parent}" prefix="${prefix}" number="2" x_loc="-0.055" y_loc= "0.120" z_loc="0.1028"/>
+    <xacro:stack_bottom_pole parent="${parent}" prefix="${prefix}" number="3" x_loc= "0.120" y_loc="-0.082" z_loc="0.1028"/>
+    <xacro:stack_bottom_pole parent="${parent}" prefix="${prefix}" number="4" x_loc= "0.055" y_loc="-0.120" z_loc="0.1028"/>
+    <xacro:stack_bottom_pole parent="${parent}" prefix="${prefix}" number="5" x_loc="-0.055" y_loc="-0.120" z_loc="0.1028"/>
+    <joint name="${prefix}/plate_bottom_joint" type="fixed">
       <origin xyz="0.02364 0.0 0.1306" rpy="0 0 0"/>
       <parent link="${parent}"/>
-      <child link="plate_bottom_link"/>
-    </joint>
-    <link name="plate_bottom_link">
+      <child link="${prefix}/plate_bottom_link"/>
+    </joint>
+    <link name="${prefix}/plate_bottom_link">
       <visual>
         <origin xyz="0 0 0" rpy="0 0 0"/>
@@ -160,14 +160,14 @@
       </inertial>
     </link>
-    <xacro:stack_middle_pole parent="${parent}" number="0" x_loc= "0.0381" y_loc= "0.1505" z_loc="0.1640"/>
-    <xacro:stack_middle_pole parent="${parent}" number="1" x_loc= "0.0381" y_loc="-0.1505" z_loc="0.1640"/>
-    <xacro:stack_middle_pole parent="${parent}" number="2" x_loc="-0.0381" y_loc= "0.1505" z_loc="0.1640"/>
-    <xacro:stack_middle_pole parent="${parent}" number="3" x_loc="-0.0381" y_loc="-0.1505" z_loc="0.1640"/>
-    <joint name="plate_middle_joint" type="fixed">
+    <xacro:stack_middle_pole parent="${parent}" prefix="${prefix}" number="0" x_loc= "0.0381" y_loc= "0.1505" z_loc="0.1640"/>
+    <xacro:stack_middle_pole parent="${parent}" prefix="${prefix}" number="1" x_loc= "0.0381" y_loc="-0.1505" z_loc="0.1640"/>
+    <xacro:stack_middle_pole parent="${parent}" prefix="${prefix}" number="2" x_loc="-0.0381" y_loc= "0.1505" z_loc="0.1640"/>
+    <xacro:stack_middle_pole parent="${parent}" prefix="${prefix}" number="3" x_loc="-0.0381" y_loc="-0.1505" z_loc="0.1640"/>
+    <joint name="${prefix}/plate_middle_joint" type="fixed">
       <origin xyz="-0.01364 0.0 0.1874" rpy="0 0 0"/>
       <parent link="${parent}"/>
-      <child link="plate_middle_link"/>
-    </joint>
-    <link name="plate_middle_link">
+      <child link="${prefix}/plate_middle_link"/>
+    </joint>
+    <link name="${prefix}/plate_middle_link">
       <visual>
         <origin xyz="0 0 0" rpy="0 0 0"/>
@@ -190,16 +190,16 @@
       </inertial>
     </link>
-    <xacro:stack_top_pole parent="${parent}" number="0" x_loc= "0.0381" y_loc= "0.1505" z_loc="0.2920"/>
-    <xacro:stack_top_pole parent="${parent}" number="1" x_loc= "0.0381" y_loc="-0.1505" z_loc="0.2920"/>
-    <xacro:stack_top_pole parent="${parent}" number="2" x_loc="-0.0381" y_loc= "0.1505" z_loc="0.2920"/>
-    <xacro:stack_top_pole parent="${parent}" number="3" x_loc="-0.0381" y_loc="-0.1505" z_loc="0.2920"/>
-    <xacro:stack_3d_sensor_pole parent="${parent}" number="0" x_loc="-0.1024" y_loc= "0.098" z_loc="0.2372"/>
-    <xacro:stack_3d_sensor_pole parent="${parent}" number="1" x_loc="-0.1024" y_loc="-0.098" z_loc="0.2372"/>
-    <joint name="plate_top_joint" type="fixed">
+    <xacro:stack_top_pole parent="${parent}" prefix="${prefix}" number="0" x_loc= "0.0381" y_loc= "0.1505" z_loc="0.2920"/>
+    <xacro:stack_top_pole parent="${parent}" prefix="${prefix}" number="1" x_loc= "0.0381" y_loc="-0.1505" z_loc="0.2920"/>
+    <xacro:stack_top_pole parent="${parent}" prefix="${prefix}" number="2" x_loc="-0.0381" y_loc= "0.1505" z_loc="0.2920"/>
+    <xacro:stack_top_pole parent="${parent}" prefix="${prefix}" number="3" x_loc="-0.0381" y_loc="-0.1505" z_loc="0.2920"/>
+    <xacro:stack_3d_sensor_pole parent="${parent}" prefix="${prefix}" number="0" x_loc="-0.1024" y_loc= "0.098" z_loc="0.2372"/>
+    <xacro:stack_3d_sensor_pole parent="${parent}" prefix="${prefix}" number="1" x_loc="-0.1024" y_loc="-0.098" z_loc="0.2372"/>
+    <joint name="${prefix}/plate_top_joint" type="fixed">
       <origin xyz="-0.01364 0.0  0.3966" rpy="0 0 0"/>
       <parent link="${parent}"/>
-      <child link="plate_top_link"/>
-    </joint>
-    <link name="plate_top_link">
+      <child link="${prefix}/plate_top_link"/>
+    </joint>
+    <link name="${prefix}/plate_top_link">
       <visual>
         <origin xyz="0 0 0" rpy="0 0 0"/>

File: scarab_description/urdf/kobuki.urdf.xacro (robot description, xacro)
@@ -1,6 +1,7 @@
 <?xml version="1.0" ?>
 <!--
-This is not a standalone urdf for kobuki. It simply defines the scarab tag that can
-be incorporated by other urdf files (e.g. turtlebot).  -->
+This is not a standalone urdf for kobuki. It simply defines the scarab tag that
+can be incorporated by other urdf files (e.g. turtlebot).
+-->
 <robot name="kobuki" xmlns:xacro="http://ros.org/wiki/xacro">
   <xacro:include filename="$(find scarab_description)/urdf/common_properties.urdf.xacro"/>
@@ -8,20 +9,18 @@
   <!-- Kobuki -->
   <xacro:macro name="kobuki">
-    <link name="base_footprint"/>
+    <link name="$(arg tf_prefix)/base_footprint"/>
     <!--
-        Base link is set at the bottom of the base mould.
-        This is done to be compatible with the way base link
-        was configured for turtlebot 1. Refer to
-https://github.com/turtlebot/turtlebot/issues/40
-To put the base link at the more oft used wheel
-axis, set the z-distance from the base_footprint
-to 0.352.
+    Base link is set at the bottom of the base mould. This is done to be
+    compatible with the way base link was configured for turtlebot 1. Refer to
+    https://github.com/turtlebot/turtlebot/issues/40
+    To put the base link at the more oft used wheel axis, set the z-distance
+    from the base_footprint to 0.352.
     -->
-    <joint name="base_joint" type="fixed">
+    <joint name="$(arg tf_prefix)/base_joint" type="fixed">
       <origin xyz="0 0 0.0102" rpy="0 0 0" />
-      <parent link="base_footprint"/>
-      <child link="base_link" />
+      <parent link="$(arg tf_prefix)/base_footprint"/>
+      <child link="$(arg tf_prefix)/base_link" />
     </joint>
-    <link name="base_link">
+    <link name="$(arg tf_prefix)/base_link">
       <visual>
         <geometry>
@@ -41,10 +40,12 @@
         <origin xyz="0.01 0 0"/>
         <mass value="2.4"/> <!-- 2.4/2.6 kg for small/big battery pack -->
-        <!-- Kobuki's inertia tensor is approximated by a cylinder with homogeneous mass distribution
-             More details: http://en.wikipedia.org/wiki/List_of_moment_of_inertia_tensors
-             m = 2.4 kg; h = 0.09 m; r = 0.175 m
-             ixx = 1/12 * m * (3 * r^2 + h^2)
-             iyy = 1/12 * m * (3 * r^2 + h^2)
-             izz = 1/2 * m * r^2
+        <!--
+        Kobuki's inertia tensor is approximated by a cylinder with homogeneous
+        mass distribution More details:
+        http://en.wikipedia.org/wiki/List_of_moment_of_inertia_tensors
+        m = 2.4 kg; h = 0.09 m; r = 0.175 m
+        ixx = 1/12 * m * (3 * r^2 + h^2)
+        iyy = 1/12 * m * (3 * r^2 + h^2)
+        izz = 1/2 * m * r^2
         -->
         <inertia ixx="0.019995" ixy="0.0" ixz="0.0"
@@ -53,11 +54,11 @@
       </inertial>
     </link>
-    <joint name="wheel_left_joint" type="continuous">
-      <parent link="base_link"/>
-      <child link="wheel_left_link"/>
+    <joint name="$(arg tf_prefix)/wheel_left_joint" type="continuous">
+      <parent link="$(arg tf_prefix)/base_link"/>
+      <child link="$(arg tf_prefix)/wheel_left_link"/>
       <origin xyz="0.00 ${0.23/2} 0.0250" rpy="${-M_PI/2} 0 0"/>
       <axis xyz="0 0 1"/>
     </joint>
-    <link name="wheel_left_link">
+    <link name="$(arg tf_prefix)/wheel_left_link">
       <visual>
         <geometry>
@@ -80,11 +81,11 @@
       </inertial>
     </link>
-    <joint name="wheel_right_joint" type="continuous">
-      <parent link="base_link"/>
-      <child link="wheel_right_link"/>
+    <joint name="$(arg tf_prefix)/wheel_right_joint" type="continuous">
+      <parent link="$(arg tf_prefix)/base_link"/>
+      <child link="$(arg tf_prefix)/wheel_right_link"/>
       <origin xyz="0.00 -${0.23/2} 0.0250" rpy="${-M_PI/2} 0 0"/>
       <axis xyz="0 0 1"/>
     </joint>
-    <link name="wheel_right_link">
+    <link name="$(arg tf_prefix)/wheel_right_link">
       <visual>
         <geometry>
@@ -107,10 +108,10 @@
       </inertial>
     </link>
-    <joint name="caster_front_joint" type="fixed">
-      <parent link="base_link"/>
-      <child link="caster_front_link"/>
+    <joint name="$(arg tf_prefix)/caster_front_joint" type="fixed">
+      <parent link="$(arg tf_prefix)/base_link"/>
+      <child link="$(arg tf_prefix)/caster_front_link"/>
       <origin xyz="0.115 0.0 0.007" rpy="${-M_PI/2} 0 0"/>
     </joint>
-    <link name="caster_front_link">
+    <link name="$(arg tf_prefix)/caster_front_link">
       <collision>
         <geometry>
@@ -127,10 +128,10 @@
       </inertial>
     </link>
-    <joint name="caster_back_joint" type="fixed">
-      <parent link="base_link"/>
-      <child link="caster_back_link"/>
+    <joint name="$(arg tf_prefix)/caster_back_joint" type="fixed">
+      <parent link="$(arg tf_prefix)/base_link"/>
+      <child link="$(arg tf_prefix)/caster_back_link"/>
       <origin xyz="-0.135 0.0 0.009" rpy="${-M_PI/2} 0 0"/>
     </joint>
-    <link name="caster_back_link">
+    <link name="$(arg tf_prefix)/caster_back_link">
       <collision>
         <geometry>

File: scarab_description/urdf/kobuki_gazebo.urdf.xacro (robot description, xacro)
@@ -2,5 +2,5 @@
 <robot name="kobuki_sim" xmlns:xacro="http://ros.org/wiki/xacro">
   <xacro:macro name="kobuki_sim">
-    <gazebo reference="wheel_left_link">
+    <gazebo reference="$(arg tf_prefix)/wheel_left_link">
       <mu1>1.0</mu1>
       <mu2>1.0</mu2>
@@ -8,5 +8,5 @@
       <kd>10000.0</kd>
     </gazebo>
-    <gazebo reference="wheel_right_link">
+    <gazebo reference="$(arg tf_prefix)/wheel_right_link">
       <mu1>1.0</mu1>
       <mu2>1.0</mu2>
@@ -14,5 +14,5 @@
       <kd>10000.0</kd>
     </gazebo>
-    <gazebo reference="caster_front_link">
+    <gazebo reference="$(arg tf_prefix)/caster_front_link">
       <mu1>0.0</mu1>
       <mu2>0.0</mu2>
@@ -20,5 +20,5 @@
       <kd>10000.0</kd>
     </gazebo>
-    <gazebo reference="caster_back_link">
+    <gazebo reference="$(arg tf_prefix)/caster_back_link">
       <mu1>0.0</mu1>
       <mu2>0.0</mu2>
@@ -26,5 +26,5 @@
       <kd>10000.0</kd>
     </gazebo>
-    <gazebo reference="base_link">
+    <gazebo reference="$(arg tf_prefix)/base_link">
       <sensor type="contact" name="bumpers">
 	      <always_on>1</always_on>
@@ -42,6 +42,6 @@
         <updateRate>10</updateRate>
         <!-- BWC: This is intentionally flipped; not sure why necessary -->
-        <leftJoint>wheel_left_joint</leftJoint>
-        <rightJoint>wheel_right_joint</rightJoint>
+        <leftJoint>$(arg tf_prefix)/wheel_left_joint</leftJoint>
+        <rightJoint>$(arg tf_prefix)/wheel_right_joint</rightJoint>
         <wheelSeparation>0.230</wheelSeparation>
         <wheelDiameter>0.070</wheelDiameter>
@@ -49,6 +49,6 @@
         <commandTopic>cmd_vel</commandTopic>
         <odometryTopic>ground_truth/odom</odometryTopic>
-        <odometryFrame>ground_truth/odom</odometryFrame>
-        <robotBaseFrame>ground_truth/base_link</robotBaseFrame>
+        <odometryFrame>$(arg tf_prefix)/ground_truth/odom</odometryFrame>
+        <robotBaseFrame>$(arg tf_prefix)/ground_truth/base_link</robotBaseFrame>
         <publishWheelJointState>false</publishWheelJointState>
         <wheelAcceleration>0</wheelAcceleration>
@@ -57,4 +57,5 @@
         <publishTf>1</publishTf>
         <publishWheelTF>false</publishWheelTF>
+        <publishOdomTF>1</publishOdomTF>
       </plugin>
     </gazebo>

File: scarab_description/urdf/scarab.xacro (robot description, xacro)
@@ -15,6 +15,6 @@
   <xacro:include filename="$(find scarab_description)/urdf/sensors/asus_xtion_pro.urdf.xacro"/>
   <xacro:kobuki/>
-  <xacro:stack_hexagons parent="base_link"/>
-  <xacro:sensor_kinect  parent="base_link"/>
+  <xacro:stack_hexagons parent="$(arg tf_prefix)/base_link" prefix="$(arg tf_prefix)"/>
+  <xacro:sensor_kinect  parent="$(arg tf_prefix)/base_link" prefix="$(arg tf_prefix)"/>
   <xacro:include filename="$(find scarab_description)/urdf/sensors/hokuyo.gazebo" />
 </robot>

File: scarab_description/urdf/sensors/asus_xtion_pro.urdf.xacro (robot description, xacro)
@@ -8,12 +8,12 @@
   <xacro:property name="asus_xtion_pro_cam_rel_rgb_py"   value="-0.0220" />
   <!-- Parameterised in part by the values in turtlebot_properties.urdf.xacro -->
-  <xacro:macro name="sensor_asus_xtion_pro" params="parent">
-    <joint name="camera_rgb_joint" type="fixed">
+  <xacro:macro name="sensor_asus_xtion_pro" params="parent prefix">
+    <joint name="${prefix}/camera_rgb_joint" type="fixed">
       <origin xyz="${cam_px} ${cam_py} ${cam_pz}"
               rpy="${cam_or} ${cam_op} ${cam_oy}"/>
       <parent link="${parent}"/>
-      <child link="camera_rgb_frame" />
+      <child link="${prefix}/camera_rgb_frame" />
     </joint>
-    <link name="camera_rgb_frame">
+    <link name="${prefix}/camera_rgb_frame">
       <inertial>
         <mass value="0.001" />
@@ -24,10 +24,10 @@
       </inertial>
     </link>
-    <joint name="camera_rgb_optical_joint" type="fixed">
+    <joint name="${prefix}/camera_rgb_optical_joint" type="fixed">
       <origin xyz="0 0 0" rpy="${-M_PI/2} 0 ${-M_PI/2}" />
-      <parent link="camera_rgb_frame" />
-      <child link="camera_rgb_optical_frame" />
+      <parent link="${prefix}/camera_rgb_frame" />
+      <child link="${prefix}/camera_rgb_optical_frame" />
     </joint>
-    <link name="camera_rgb_optical_frame">
+    <link name="${prefix}/camera_rgb_optical_frame">
       <inertial>
         <mass value="0.001" />
@@ -38,11 +38,11 @@
       </inertial>
     </link>
-    <joint name="camera_joint" type="fixed">
+    <joint name="${prefix}/camera_joint" type="fixed">
       <origin xyz="0 ${asus_xtion_pro_cam_rel_rgb_py} 0"
               rpy="0 0 0"/>
-      <parent link="camera_rgb_frame"/>
-      <child link="camera_link"/>
+      <parent link="${prefix}/camera_rgb_frame"/>
+      <child link="${prefix}/camera_link"/>
     </joint>
-    <link name="camera_link">
+    <link name="${prefix}/camera_link">
       <visual>
         <origin xyz="-0.01 0 0" rpy="${-M_PI/2} -${M_PI} ${-M_PI/2}"/>
@@ -65,10 +65,10 @@
       </inertial>
     </link>
-    <joint name="camera_depth_joint" type="fixed">
+    <joint name="${prefix}/camera_depth_joint" type="fixed">
       <origin xyz="0 ${asus_xtion_pro_depth_rel_rgb_py} 0" rpy="0 0 0" />
-      <parent link="camera_rgb_frame" />
-      <child link="camera_depth_frame" />
+      <parent link="${prefix}/camera_rgb_frame" />
+      <child link="${prefix}/camera_depth_frame" />
     </joint>
-    <link name="camera_depth_frame">
+    <link name="${prefix}/camera_depth_frame">
       <inertial>
         <mass value="0.01" />
@@ -79,10 +79,10 @@
       </inertial>
     </link>
-    <joint name="camera_depth_optical_joint" type="fixed">
+    <joint name="${prefix}/camera_depth_optical_joint" type="fixed">
       <origin xyz="0 0 0" rpy="${-M_PI/2} 0 ${-M_PI/2}" />
-      <parent link="camera_depth_frame" />
-      <child link="camera_depth_optical_frame" />
+      <parent link="${prefix}/camera_depth_frame" />
+      <child link="${prefix}/camera_depth_optical_frame" />
     </joint>
-    <link name="camera_depth_optical_frame">
+    <link name="${prefix}/camera_depth_optical_frame">
       <inertial>
         <mass value="0.001" />
