Commit message: enable multi-scarab gazebo simulations
1) added tf_prefix throughout scarab description files to avoid tf collisions
2) updated scarab_sim.launch file to work with update tf tree
3) added PERCH environment

File: scarab_description/urdf/sensors/kinect.urdf.xacro (robot description, xacro)
@@ -4,11 +4,11 @@
   <xacro:include filename="$(find scarab_description)/urdf/turtlebot_properties.urdf.xacro"/>
   <!-- Parameterised in part by the values in turtlebot_properties.urdf.xacro -->
-  <xacro:macro name="sensor_kinect" params="parent">
-    <joint name="camera_rgb_joint" type="fixed">
+  <xacro:macro name="sensor_kinect" params="parent prefix">
+    <joint name="${prefix}/camera_rgb_joint" type="fixed">
       <origin xyz="${cam_px} ${cam_py} ${cam_pz}" rpy="${cam_or} ${cam_op} ${cam_oy}"/>
       <parent link="${parent}"/>
-      <child link="camera_rgb_frame" />
+      <child link="${prefix}/camera_rgb_frame" />
     </joint>
-    <link name="camera_rgb_frame">
+    <link name="${prefix}/camera_rgb_frame">
       <inertial>
         <mass value="0.001" />
@@ -19,10 +19,10 @@
       </inertial>
     </link>
-    <joint name="camera_rgb_optical_joint" type="fixed">
+    <joint name="${prefix}/camera_rgb_optical_joint" type="fixed">
       <origin xyz="0 0 0" rpy="${-M_PI/2} 0 ${-M_PI/2}" />
-      <parent link="camera_rgb_frame" />
-      <child link="camera_rgb_optical_frame" />
+      <parent link="${prefix}/camera_rgb_frame" />
+      <child link="${prefix}/camera_rgb_optical_frame" />
     </joint>
-    <link name="camera_rgb_optical_frame">
+    <link name="${prefix}/camera_rgb_optical_frame">
       <inertial>
         <mass value="0.001" />
@@ -33,63 +33,63 @@
       </inertial>
     </link>
-  <joint name="camera_joint" type="fixed">
-    <origin xyz="-0.031 ${-cam_py} -0.016" rpy="0 0 0"/>
-    <parent link="camera_rgb_frame"/>
-    <child link="camera_link"/>
-  </joint>
-    <link name="camera_link">
-    <visual>
-     <origin xyz="0 0 0" rpy="0 0 ${M_PI/2}"/>
-      <geometry>
-       <mesh filename="package://scarab_description/meshes/sensors/kinect.dae"/>
-      </geometry>
-    </visual>
-	  <collision>
-      <origin xyz="0.0 0.0 0.0" rpy="0 0 0"/>
-	    <geometry>
-	      <box size="0.07271 0.27794 0.073"/>
-	    </geometry>
-	  </collision>
-    <inertial>
-      <mass value="0.001" />
-      <origin xyz="0 0 0" />
-      <inertia ixx="0.0001" ixy="0.0" ixz="0.0"
-               iyy="0.0001" iyz="0.0"
-               izz="0.0001" />
-    </inertial>
-  </link>
-  <!-- The fixed joints & links below are usually published by static_transformers launched by the OpenNi launch
-       files. However, for Gazebo simulation we need them, so we add them here.
-       (Hence, don't publish them additionally!) -->
-	<joint name="camera_depth_joint" type="fixed">
-	  <origin xyz="0 ${2 * -cam_py} 0" rpy="0 0 0" />
-	  <parent link="camera_rgb_frame" />
-	  <child link="camera_depth_frame" />
-	</joint>
-	<link name="camera_depth_frame">
-    <inertial>
-      <mass value="0.001" />
-      <origin xyz="0 0 0" />
-      <inertia ixx="0.0001" ixy="0.0" ixz="0.0"
-               iyy="0.0001" iyz="0.0"
-               izz="0.0001" />
-    </inertial>
-	</link>
-	<joint name="camera_depth_optical_joint" type="fixed">
-	  <origin xyz="0 0 0" rpy="${-M_PI/2} 0 ${-M_PI/2}" />
-	  <parent link="camera_depth_frame" />
-	  <child link="camera_depth_optical_frame" />
-	</joint>
-	<link name="camera_depth_optical_frame">
-    <inertial>
-      <mass value="0.001" />
-      <origin xyz="0 0 0" />
-      <inertia ixx="0.0001" ixy="0.0" ixz="0.0"
-               iyy="0.0001" iyz="0.0"
-               izz="0.0001" />
-    </inertial>
-	</link>
-	<!-- Kinect sensor for simulation -->
-	<xacro:turtlebot_sim_3dsensor/>
+    <joint name="${prefix}/camera_joint" type="fixed">
+      <origin xyz="-0.031 ${-cam_py} -0.016" rpy="0 0 0"/>
+      <parent link="${prefix}/camera_rgb_frame"/>
+      <child link="${prefix}/camera_link"/>
+    </joint>
+    <link name="${prefix}/camera_link">
+      <visual>
+        <origin xyz="0 0 0" rpy="0 0 ${M_PI/2}"/>
+        <geometry>
+          <mesh filename="package://scarab_description/meshes/sensors/kinect.dae"/>
+        </geometry>
+      </visual>
+      <collision>
+        <origin xyz="0.0 0.0 0.0" rpy="0 0 0"/>
+        <geometry>
+          <box size="0.07271 0.27794 0.073"/>
+        </geometry>
+      </collision>
+      <inertial>
+        <mass value="0.001" />
+        <origin xyz="0 0 0" />
+        <inertia ixx="0.0001" ixy="0.0" ixz="0.0"
+                 iyy="0.0001" iyz="0.0"
+                 izz="0.0001" />
+      </inertial>
+    </link>
+    <!-- The fixed joints & links below are usually published by static_transformers launched by the OpenNi launch
+         files. However, for Gazebo simulation we need them, so we add them here.
+         (Hence, don't publish them additionally!) -->
+    <joint name="${prefix}/camera_depth_joint" type="fixed">
+      <origin xyz="0 ${2 * -cam_py} 0" rpy="0 0 0" />
+      <parent link="${prefix}/camera_rgb_frame" />
+      <child link="${prefix}/camera_depth_frame" />
+    </joint>
+    <link name="${prefix}/camera_depth_frame">
+      <inertial>
+        <mass value="0.001" />
+        <origin xyz="0 0 0" />
+        <inertia ixx="0.0001" ixy="0.0" ixz="0.0"
+                 iyy="0.0001" iyz="0.0"
+                 izz="0.0001" />
+      </inertial>
+    </link>
+    <joint name="${prefix}/camera_depth_optical_joint" type="fixed">
+      <origin xyz="0 0 0" rpy="${-M_PI/2} 0 ${-M_PI/2}" />
+      <parent link="${prefix}/camera_depth_frame" />
+      <child link="${prefix}/camera_depth_optical_frame" />
+    </joint>
+    <link name="${prefix}/camera_depth_optical_frame">
+      <inertial>
+        <mass value="0.001" />
+        <origin xyz="0 0 0" />
+        <inertia ixx="0.0001" ixy="0.0" ixz="0.0"
+                 iyy="0.0001" iyz="0.0"
+                 izz="0.0001" />
+      </inertial>
+    </link>
+    <!-- Kinect sensor for simulation -->
+    <xacro:turtlebot_sim_3dsensor/>
   </xacro:macro>
 </robot>

File: scarab_description/urdf/turtlebot_gazebo.urdf.xacro (robot description, xacro)
@@ -3,5 +3,5 @@
   <!-- Microsoft Kinect / ASUS Xtion PRO Live for simulation -->
   <xacro:macro name="turtlebot_sim_3dsensor">
-    <gazebo reference="camera_link">
+    <gazebo reference="$(arg tf_prefix)/camera_link">
       <sensor type="depth" name="camera">
         <always_on>true</always_on>
@@ -28,5 +28,5 @@
           <cameraInfoTopicName>rgb/camera_info</cameraInfoTopicName>
           <depthImageCameraInfoTopicName>depth/camera_info</depthImageCameraInfoTopicName>
-          <frameName>camera_depth_optical_frame</frameName>
+          <frameName>$(arg tf_prefix)/camera_depth_optical_frame</frameName>
           <distortion_k1>0.0</distortion_k1>
           <distortion_k2>0.0</distortion_k2>

File: scarab_description/urdf/turtlebot_properties.urdf.xacro (robot description, xacro)
@@ -19,9 +19,9 @@
      (currently in development and awaiting feedback)
    -->
-	<xacro:property name="cam_px" value="-0.0" />
-	<xacro:property name="cam_py" value="-0.0" />
-	<xacro:property name="cam_pz" value="0.3" />
-	<xacro:property name="cam_or" value="0" />
-	<xacro:property name="cam_op" value="-0.357" />
-	<xacro:property name="cam_oy" value="0" />
+  <xacro:property name="cam_px" value="-0.0" />
+  <xacro:property name="cam_py" value="-0.0" />
+  <xacro:property name="cam_pz" value="0.3" />
+  <xacro:property name="cam_or" value="0" />
+  <xacro:property name="cam_op" value="-0.357" />
+  <xacro:property name="cam_oy" value="0" />
 </robot>
