Commit message: Modify scarab model to point camera forward

File: scarab_description/urdf/scarab.xacro (robot description, xacro)
@@ -15,5 +15,5 @@
   <!-- 3D Sensors -->
   <xacro:include filename="$(find scarab_description)/urdf/sensors/kinect.urdf.xacro"/>
-  <xacro:include filename="$(find scarab_description)/urdf/sensors/asus_xtion_pro.urdf.xacro"/>
+  <!-- <xacro:include filename="$(find scarab_description)/urdf/sensors/asus_xtion_pro.urdf.xacro"/> -->
   <xacro:kobuki/>
   <xacro:stack_hexagons parent="$(arg tf_prefix)/base_link" prefix="$(arg tf_prefix)"/>

File: scarab_description/urdf/sensors/asus_xtion_pro.urdf.xacro (robot description, xacro)
@@ -25,5 +25,5 @@
     </link>
     <joint name="${prefix}/camera_rgb_optical_joint" type="fixed">
-      <origin xyz="0 0 0" rpy="${-M_PI/2} 0 ${-M_PI/2}" />
+      <origin xyz="0 0 0" rpy="${-M_PI/2} 0 ${-M_PI/2}" />z
       <parent link="${prefix}/camera_rgb_frame" />
       <child link="${prefix}/camera_rgb_optical_frame" />

File: scarab_description/urdf/turtlebot_gazebo.urdf.xacro (robot description, xacro)
@@ -6,5 +6,5 @@
       <sensor type="depth" name="camera">
         <always_on>true</always_on>
-        <update_rate>5</update_rate>
+        <update_rate>20</update_rate>
         <camera>
           <horizontal_fov>${60.0*M_PI/180.0}</horizontal_fov>
@@ -16,5 +16,5 @@
           <clip>
             <near>0.1</near>
-            <far>50.0</far>
+            <far>5.0</far>
           </clip>
         </camera>
@@ -22,5 +22,5 @@
           <cameraName>camera</cameraName>
           <alwaysOn>true</alwaysOn>
-          <updateRate>5</updateRate>
+          <updateRate>20</updateRate>
           <imageTopicName>rgb/image_raw</imageTopicName>
           <depthImageTopicName>depth/image_raw</depthImageTopicName>
@@ -34,6 +34,6 @@
           <distortion_t1>0.0</distortion_t1>
           <distortion_t2>0.0</distortion_t2>
-          <pointCloudCutoff>0.4</pointCloudCutoff>
-          <pointCloudCutoffMax>50.0</pointCloudCutoffMax>
+          <pointCloudCutoff>0.1</pointCloudCutoff>
+          <pointCloudCutoffMax>5.0</pointCloudCutoffMax>
         </plugin>
       </sensor>

File: scarab_description/urdf/turtlebot_properties.urdf.xacro (robot description, xacro)
@@ -23,5 +23,6 @@
   <xacro:property name="cam_pz" value="0.3" />
   <xacro:property name="cam_or" value="0" />
-  <xacro:property name="cam_op" value="-0.357" />
+  <!-- <xacro:property name="cam_op" value="-0.357" /> -->
+  <xacro:property name="cam_op" value="0" />
   <xacro:property name="cam_oy" value="0" />
 </robot>
